File: Alarm-clock-v2/Alarm-clock-v2.sch (KiCad schematic (older format))
At the start: 23 parts, among them CON1 AVR-ISP-6, J1 USB_OTG, SW1 SW_SPST, SW2 SW_SPST, SW3 SW_SPST, U1 ATMEGA32U4-AU, U2 CA56-12CGKWA, Y1 Crystal

Commit message: Added buzzer
Parts:
- added BZ1: Buzzer, Buzzers_Beepers:BUZZER, symbol Buzzer
Connections:
- wire segments 96 -> 99
- no-connect marks 9 -> 8
Changed lines of the file:
@@
 LIBS:contrib
 LIBS:valves
+LIBS:Alarm-clock-v2-cache
 EELAYER 25 0
 EELAYER END
@@
 NoConn ~ 5200 4250
 NoConn ~ 5200 4350
-NoConn ~ 5200 4550
 NoConn ~ 5200 5050
 NoConn ~ 2950 5250
@@
 Text Label 5250 4750 0    60   ~ 0
 DIGIT1
+$Comp
+L Buzzer BZ1
+U 1 1 5A997B30
+P 6200 4650
+F 0 "BZ1" H 6350 4700 50  0000 L CNN
+F 1 "Buzzer" H 6350 4600 50  0000 L CNN
+F 2 "Buzzers_Beepers:BUZZER" V 6175 4750 50  0001 C CNN
+F 3 "" V 6175 4750 50  0001 C CNN
+	1    6200 4650
+	1    0    0    -1
+$EndComp
+Wire Wire Line
+	5200 4550 6100 4550
+$Comp
+L GND #PWR014
+U 1 1 5A997C88
+P 6000 4850
+F 0 "#PWR014" H 6000 4600 50  0001 C CNN
+F 1 "GND" H 6000 4700 50  0000 C CNN
+F 2 "" H 6000 4850 50  0001 C CNN
+F 3 "" H 6000 4850 50  0001 C CNN
+	1    6000 4850
+	1    0    0    -1
+$EndComp
+Wire Wire Line
+	6000 4850 6000 4750
+Wire Wire Line
+	6000 4750 6100 4750
 $EndSCHEMATC
